File: hardware/overlay64.sch (KiCad schematic (older format))
At the start: 26 parts, among them IC1 ATMEGA1284, P1 USB, P2 INPUT, P3 CONTROL, P4 MAIN, P5 HOLE, P6 HOLE, P7 HOLE, P8 HOLE, P9 BYPASS, SW1 SW_BOOT, U1 LM1881, Y1 20MHz

Commit message: Project: Hardware documentation licensed under CERN OHL 1.2
Other:
- note added: "Overlay64 video overlay module\nCopyright 2016 Henning Bekel\n\nThis documentation describes Open Hardware and is \nlicensed under the CERN OHL v. 1.2.\n\nYou may redistribute and modify this documentation\nunder the terms of the CERN OHL v.1.2. (http://ohwr.org/cernohl).\nThis documentation is distributed WITHOUT ANY EXPRESS OR \nIMPLIED WARRANTY, INCLUDING OF MERCHANTABILITY, \nSATISFACTORY QUA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"
- moved on the sheet: SW1
Changed lines of the file:
@@
 encoding utf-8
 Sheet 1 1
-Title "Simple Video Overlay Driver"
+Title "Overlay64 -- Video Overlay Module"
 Date "2016-02-02"
 Rev "1"
 Comp "Henning Bekel"
-Comment1 "http://www.henning-bekel.de"
-Comment2 ""
+Comment1 "http://www.henning-bekel.de/overlay64"
+Comment2 "Licensed under CERN OHL v.1.2"
 Comment3 ""
 Comment4 ""
@@
 L GND #PWR024
 U 1 1 57B5BBC8
-P 2750 6350
-F 0 "#PWR024" H 2750 6100 50  0001 C CNN
-F 1 "GND" H 2750 6200 50  0000 C CNN
-F 2 "" H 2750 6350 50  0000 C CNN
-F 3 "" H 2750 6350 50  0000 C CNN
-	1    2750 6350
-	1    0    0    -1
-$EndComp
-Text Label 3050 6350 0    60   ~ 0
+P 1100 4200
+F 0 "#PWR024" H 1100 3950 50  0001 C CNN
+F 1 "GND" H 1100 4050 50  0000 C CNN
+F 2 "" H 1100 4200 50  0000 C CNN
+F 3 "" H 1100 4200 50  0000 C CNN
+	1    1100 4200
+	1    0    0    -1
+$EndComp
+Text Label 1400 4200 0    60   ~ 0
 BOOT
 NoConn ~ 2000 1800
@@
 L SW_PUSH_SMALL_H SW1
 U 1 1 5832A426
-P 2900 6350
-F 0 "SW1" H 2980 6460 50  0000 C CNN
-F 1 "SW_BOOT" H 3260 6290 50  0000 C CNN
-F 2 "custom:Button" H 2900 6550 50  0001 C CNN
-F 3 "" H 2900 6550 50  0000 C CNN
-	1    2900 6350
-	1    0    0    -1
-$EndComp
+P 1250 4200
+F 0 "SW1" H 1330 4310 50  0000 C CNN
+F 1 "SW_BOOT" H 1610 4140 50  0000 C CNN
+F 2 "custom:Button" H 1250 4400 50  0001 C CNN
+F 3 "" H 1250 4400 50  0000 C CNN
+	1    1250 4200
+	1    0    0    -1
+$EndComp
+Text Notes 600  7700 0    60   ~ 0
+Overlay64 video overlay module\nCopyright 2016 Henning Bekel\n\nThis documentation describes Open Hardware and is \nlicensed under the CERN OHL v. 1.2.\n\nYou may redistribute and modify this documentation\nunder the terms of the CERN OHL v.1.2. (http://ohwr.org/cernohl).\nThis documentation is distributed WITHOUT ANY EXPRESS OR \nIMPLIED WARRANTY, INCLUDING OF MERCHANTABILITY, \nSATISFACTORY QUALITY AND FITNESS FOR A PARTICULAR \nPURPOSE. Please see the CERN OHL v.1.2 for applicable conditions
 $EndSCHEMATC
